File: KiCad/KiCad.kicad_sch (KiCad schematic)
At the start: 16 parts, among them M1 Servo (SG90), U1 ESP32-DEVKITC, U2 microSD-DIP-KIT

Commit message: 余計なものを削除
Parts:
- removed D2, D3, D4, D5: LED, LED_THT:LED_D5.0mm, symbol Device:LED
- removed M1: Servo (SG90), Connector_PinHeader_2.54mm:PinHeader_1x03_P2.54mm_Horizontal, symbol Motor:Motor_Servo
- removed R2, R3, R4, R5: 330, Resistor_THT:R_Axial_DIN0204_L3.6mm_D1.6mm_P5.08mm_Horizontal, symbol Device:R
Connections:
- net GND: no longer U1.14 (GND1)
- no-connect marks 22 -> 28
